File: Hardware/mushroom_pcb.kicad_sch (KiCad schematic)
At the start: 52 parts, among them J1 Conn_01x04, J2 Conn_01x07_Pin, J3 Screw_Terminal_01x03, J4 Screw_Terminal_01x02, J5 Screw_Terminal_01x02, J6 Screw_Terminal_01x03, J7 Conn_01x03_Pin, J8 Conn_01x04_Pin, J9 Barrel_Jack, Q3 AO3400A, Q4 AO3400A, SW1 SW_Push, SW2 SW_Push, SW3 RotaryEncoder_Switch, U1 ESP32-WROOM-32E, U2 LM2596S-5, U3 ME6211C33M5

Commit message: Nueva version más compacta y con elementos handsoldering (falta rutear y cambiar algunas huellas)
Parts:
- R1: footprint Resistor_SMD:R_0508_1220Metric -> Resistor_SMD:R_0805_2012Metric_Pad1.20x1.40mm_HandSolder
- R10, R11, R12, R13, R14, R15, R5, R6, R7, R8, R9: footprint Resistor_SMD:R_0805_2012Metric -> Resistor_SMD:R_0805_2012Metric_Pad1.20x1.40mm_HandSolder
- R2, R3, R4: footprint Resistor_SMD:R_0603_1608Metric -> Resistor_SMD:R_0805_2012Metric_Pad1.20x1.40mm_HandSolder
Changed lines of the file:
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@@
 			)
 		)
-		(property "Footprint" "Resistor_SMD:R_0603_1608Metric"
+		(property "Footprint" "Resistor_SMD:R_0805_2012Metric_Pad1.20x1.40mm_HandSolder"
 			(at 103.632 115.57 90)
 			(hide yes)
@@
 			)
 		)
-		(property "Footprint" "Resistor_SMD:R_0508_1220Metric"
+		(property "Footprint" "Resistor_SMD:R_0805_2012Metric_Pad1.20x1.40mm_HandSolder"
 			(at 66.04 57.912 90)
 			(hide yes)
@@
 			)
 		)
-		(property "Footprint" "Resistor_SMD:R_0603_1608Metric"
+		(property "Footprint" "Resistor_SMD:R_0805_2012Metric_Pad1.20x1.40mm_HandSolder"
 			(at 111.252 115.57 90)
 			(hide yes)
@@
 			)
 		)
-		(property "Footprint" "Resistor_SMD:R_0805_2012Metric"
+		(property "Footprint" "Resistor_SMD:R_0805_2012Metric_Pad1.20x1.40mm_HandSolder"
 			(at 21.082 171.45 90)
 			(hide yes)
@@
 			)
 		)
-		(property "Footprint" "Resistor_SMD:R_0805_2012Metric"
+		(property "Footprint" "Resistor_SMD:R_0805_2012Metric_Pad1.20x1.40mm_HandSolder"
 			(at 167.64 81.788 90)
 			(hide yes)
@@
 			)
 		)
-		(property "Footprint" "Resistor_SMD:R_0805_2012Metric"
+		(property "Footprint" "Resistor_SMD:R_0805_2012Metric_Pad1.20x1.40mm_HandSolder"
 			(at 199.39 145.288 90)
 			(hide yes)
@@
 			)
 		)
-		(property "Footprint" "Resistor_SMD:R_0805_2012Metric"
+		(property "Footprint" "Resistor_SMD:R_0805_2012Metric_Pad1.20x1.40mm_HandSolder"
 			(at 66.802 172.72 90)
 			(hide yes)
@@
 			)
 		)
-		(property "Footprint" "Resistor_SMD:R_0805_2012Metric"
+		(property "Footprint" "Resistor_SMD:R_0805_2012Metric_Pad1.20x1.40mm_HandSolder"
 			(at 201.422 118.11 90)
 			(hide yes)
@@
 			)
 		)
-		(property "Footprint" "Resistor_SMD:R_0805_2012Metric"
+		(property "Footprint" "Resistor_SMD:R_0805_2012Metric_Pad1.20x1.40mm_HandSolder"
 			(at 202.692 151.13 90)
 			(hide yes)
@@
 			)
 		)
-		(property "Footprint" "Resistor_SMD:R_0805_2012Metric"
+		(property "Footprint" "Resistor_SMD:R_0805_2012Metric_Pad1.20x1.40mm_HandSolder"
 			(at 198.12 112.268 90)
 			(hide yes)
@@
 			)
 		)
-		(property "Footprint" "Resistor_SMD:R_0805_2012Metric"
+		(property "Footprint" "Resistor_SMD:R_0805_2012Metric_Pad1.20x1.40mm_HandSolder"
 			(at 50.292 171.45 90)
 			(hide yes)
@@
 			)
 		)
-		(property "Footprint" "Resistor_SMD:R_0805_2012Metric"
+		(property "Footprint" "Resistor_SMD:R_0805_2012Metric_Pad1.20x1.40mm_HandSolder"
 			(at 80.772 172.72 90)
 			(hide yes)
@@
 			)
 		)
-		(property "Footprint" "Resistor_SMD:R_0603_1608Metric"
+		(property "Footprint" "Resistor_SMD:R_0805_2012Metric_Pad1.20x1.40mm_HandSolder"
 			(at 140.462 120.65 90)
 			(hide yes)
@@
 			)
 		)
-		(property "Footprint" "Resistor_SMD:R_0805_2012Metric"
+		(property "Footprint" "Resistor_SMD:R_0805_2012Metric_Pad1.20x1.40mm_HandSolder"
 			(at 237.49 30.988 90)
 			(hide yes)
@@
 			)
 		)
-		(property "Footprint" "Resistor_SMD:R_0805_2012Metric"
+		(property "Footprint" "Resistor_SMD:R_0805_2012Metric_Pad1.20x1.40mm_HandSolder"
 			(at 35.052 171.45 90)
 			(hide yes)

Commit message: Re ruteo placa
Connections:
- net BLK: now also U1.36 (IO22); no longer U1.23 (IO15)
- net BLOW: now also U1.8 (IO32); no longer U1.9 (IO33)
- net DC: now also U1.37 (IO23); no longer U1.24 (IO2)
- net FAN: now also U1.9 (IO33); no longer U1.8 (IO32)
- net HUM: now also U1.23 (IO15); no longer U1.36 (IO22)
- net LED: now also U1.24 (IO2); no longer U1.37 (IO23)
- net SCL: now also U1.33 (IO21); no longer U1.30 (IO18)
- net SDA: now also U1.30 (IO18); no longer U1.33 (IO21)

Commit message: cambio de conectores + octoacoplador calentador
Parts:
- removed J3, J6: Screw_Terminal_01x03, TerminalBlock_Altech:Altech_AK100_1x03_P5.00mm, symbol Connector:Screw_Terminal_01x03
- removed J4: Screw_Terminal_01x02, TerminalBlock_Altech:Altech_AK100_1x02_P5.00mm, symbol Connector:Screw_Terminal_01x02
- added J10: Screw_Terminal_01x03, TerminalBlock_Phoenix:TerminalBlock_Phoenix_PT-1,5-3-5.0-H_1x03_P5.00mm_Horizontal, symbol Connector:Screw_Terminal_01x03
- added J3, J6: Screw_Terminal_01x02, TerminalBlock_Phoenix:TerminalBlock_Phoenix_PT-1,5-2-5.0-H_1x02_P5.00mm_Horizontal, symbol Connector:Screw_Terminal_01x02
- added R16: 680, Resistor_SMD:R_0805_2012Metric_Pad1.20x1.40mm_HandSolder, symbol Device:R
- added U4: PC817, Package_DIP:DIP-4_W7.62mm, symbol Isolator:PC817
- J5: footprint TerminalBlock_Altech:Altech_AK100_1x02_P5.00mm -> TerminalBlock_Phoenix:TerminalBlock_Phoenix_PT-1,5-2-5.0-H_1x02_P5.00mm_Horizontal
- R7, R9: value R -> 10k
Connections:
- net +12V: now also J10.1 (Pin_1), J6.1 (Pin_1)
- net GND: now also J10.3 (Pin_3), J6.2 (Pin_2), U4.2
- net HEAT: now also R16.1
- net at R5.2: now also J10.2 (Pin_2)
- new net: J3.1 (Pin_1), U4.4
- new net: J3.2 (Pin_2), U4.3
- new net: R16.2, U4.1

Commit message: cambios menores, conectores + octo
Parts:
- J9: footprint Connector_BarrelJack:BarrelJack_SwitchcraftConxall_RAPC10U_Horizontal -> Connector_BarrelJack:BarrelJack_CUI_PJ-102AH_Horizontal
Changed lines of the file:
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@@
 			)
 		)
-		(property "Footprint" "Connector_BarrelJack:BarrelJack_SwitchcraftConxall_RAPC10U_Horizontal"
+		(property "Footprint" "Connector_BarrelJack:BarrelJack_CUI_PJ-102AH_Horizontal"
 			(at 130.81 61.976 0)
 			(hide yes)

Commit message: Cambios en arch de fabricacion
Parts:
- removed D1: PMEG040V050EPD, Package_TO_SOT_SMD:Nexperia_CFP15_SOT-1289, symbol Diode:PMEG040V050EPD
- added D9: SS54, Diode_SMD:D_SMA, symbol Diode:SS14
- C1, C10, C11, C2, C3, C4, C5, C6, C7, C8, C9, D2, D3, D4, D5, D6, D7, D8, J1, J10, J2, J3, J5, J6, J7, J8, J9, Q3, Q4, R1, R10, R11, R12, R13, R14, R15, R16, R2, R3, R4, R5, R6, R7, R8, R9, SW1, SW2, SW3, U4: now not fitted
Connections:
- net GND: now also D9.2 (A)
- net at L1.1, U2.2 (OUT): now also D9.1 (K)
