File: Hardware/_autosave-mushroom_pcb.kicad_sch (KiCad schematic)
At the start: 54 parts, among them J1 Conn_01x04, J10 Screw_Terminal_01x03, J2 Conn_01x07_Pin, J3 Screw_Terminal_01x02, J5 Screw_Terminal_01x02, J6 Screw_Terminal_01x02, J7 Conn_01x03_Pin, J8 Conn_01x04_Pin, J9 Barrel_Jack, Q3 AO3400A, Q4 AO3400A, SW1 SW_Push, SW2 SW_Push, SW3 RotaryEncoder_Switch, U1 ESP32-WROOM-32E, U2 LM2596S-5, U3 ME6211C33M5, U4 PC817

Commit message: version enviada a jlc
Parts:
- L1: now not fitted
Changed lines of the file:
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@@
 		(on_board yes)
 		(in_pos_files yes)
-		(dnp no)
+		(dnp yes)
 		(property "Reference" "L1"
 			(at 168.91 35.56 90)
